Commit message: changes made

File: car_description/urdf/base.urdf (robot description, URDF)
Before this commit: robot diffBase, 7 links, 6 joints
Links:
- added link base_footprint; collision box size=0.3 0.2 0.05; visual box size=0.3 0.2 0.05
Joints:
- added joint base_footprint_joint: type fixed, parent base_link, child base_footprint, origin xyz=0 0 0 rpy=0 0 0 

Commit message: Initial Commit

File: car_description/urdf/base.urdf (robot description, URDF)
Before this commit: robot car, 8 links, 7 joints
Links:
- removed link base_footprint
Joints:
- removed joint base_footprint_joint
- joint left_back_wheel_joint: axis 0 0 1 -> 0 1 0; origin xyz=-0.1 0.125 0 rpy=-1.57075 0 0 -> xyz=-0.1 0.125 0 rpy=0 0 0
- joint left_front_wheel_joint: axis 0 0 1 -> 0 1 0; origin xyz=0.1 0.125 0 rpy=-1.57075 0 0 -> xyz=0.1 0.125 0 rpy=0 0 0
- joint right_back_wheel_joint: axis 0 0 1 -> 0 1 0; origin xyz=-0.1 -0.125 0 rpy=1.57075 0 0 -> xyz=-0.1 -0.125 0 rpy=0 0 0
- joint right_front_wheel_joint: axis 0 0 1 -> 0 1 0; origin xyz=0.1 -0.125 0 rpy=1.57075 0 0 -> xyz=0.1 -0.125 0 rpy=0 0 0
